File: 01_Pcb/KY-037/KY-037/KY-037.kicad_pcb (KiCad board)
At the start: 2 copper layers, 60 x 35.5 mm, 16 parts, among them J1 Conn_01x04, Q1 2N5457, U2 LM393NG

Commit message: document
Routing:
- net Net-(U2-IN_A): track 79.5 -> 80.4 mm
Changed lines of the file:
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@@
 			(at 0.5 -3 0)
 			(layer "F.SilkS")
+			(hide yes)
 			(effects
 				(font
@@
 			(at 0 -2.75 0)
 			(layer "F.SilkS")
+			(hide yes)
 			(effects
 				(font
@@
 			(at -1 -3.5 0)
 			(layer "F.SilkS")
+			(hide yes)
 			(effects
 				(font
@@
 			(at 4 -2.5 0)
 			(layer "F.SilkS")
+			(hide yes)
 			(effects
 				(font
@@
 	)
 	(segment
-		(start 43.52 42.12)
-		(end 43.52 43.769182)
+		(start 63.088182 48.799)
+		(end 65.953818 48.799)
 		(width 0.5)
 		(layer "F.Cu")
@@
 	)
 	(segment
-		(start 50.501818 50.751)
-		(end 58.999818 50.751)
+		(start 60.750818 49)
+		(end 60.769 49)
+		(width 0.5)
+		(layer "F.Cu")
+		(net 6)
+	)
+	(segment
+		(start 58.999818 50.751)
+		(end 60.750818 49)
 		(width 0.5)
 		(layer "F.Cu")
@@
 	)
 	(segment
-		(start 66.255409 48.244591)
-		(end 66.381818 48.371)
+		(start 62.538182 48.249)
+		(end 63.088182 48.799)
 		(width 0.5)
 		(layer "F.Cu")
@@
 	)
 	(segment
-		(start 58.999818 50.751)
-		(end 61.506227 48.244591)
+		(start 50.501818 50.751)
+		(end 58.999818 50.751)
+		(width 0.5)
+		(layer "F.Cu")
+		(net 6)
+	)
+	(segment
+		(start 66.381818 48.371)
+		(end 68.189 48.371)
+		(width 0.5)
+		(layer "F.Cu")
+		(net 6)
+	)
+	(segment
+		(start 43.52 43.769182)
+		(end 50.501818 50.751)
+		(width 0.5)
+		(layer "F.Cu")
+		(net 6)
+	)
+	(segment
+		(start 60.769 48.981818)
+		(end 61.501818 48.249)
 		(width 0.5)
 		(layer "F.Cu")
@@
 	)
 	(segment
-		(start 61.506227 48.244591)
-		(end 66.255409 48.244591)
+		(start 61.501818 48.249)
+		(end 62.538182 48.249)
 		(width 0.5)
 		(layer "F.Cu")
@@
 	)
 	(segment
-		(start 66.381818 48.371)
-		(end 68.189 48.371)
+		(start 60.769 49)
+		(end 60.769 48.981818)
 		(width 0.5)
 		(layer "F.Cu")
@@
 	)
 	(segment
-		(start 43.52 43.769182)
-		(end 50.501818 50.751)
+		(start 65.953818 48.799)
+		(end 66.381818 48.371)
+		(width 0.5)
+		(layer "F.Cu")
+		(net 6)
+	)
+	(segment
+		(start 43.52 42.12)
+		(end 43.52 43.769182)
 		(width 0.5)
 		(layer "F.Cu")
@@
 	)
 	(segment
+		(start 66.56 44.24)
+		(end 67.24 44.24)
+		(width 0.5)
+		(layer "F.Cu")
+		(net 9)
+	)
+	(segment
 		(start 88.02 43.5)
 		(end 89.15137 43.5)
@@
 	)
 	(segment
+		(start 66.41 44.09)
+		(end 66.9 44.58)
+		(width 0.5)
+		(layer "F.Cu")
+		(net 9)
+	)
+	(segment
 		(start 66.9 44.58)
-		(end 71.98 39.5)
+		(end 67.24 44.24)
 		(width 0.5)
 		(layer "F.Cu")
@@
 	)
 	(segment
+		(start 66.41 44.09)
+		(end 66.56 44.24)
+		(width 0.5)
+		(layer "F.Cu")
+		(net 9)
+	)
+	(segment
+		(start 67.24 44.24)
+		(end 71.98 39.5)
+		(width 0.5)
+		(layer "F.Cu")
+		(net 9)
+	)
+	(segment
 		(start 51.02 28.7)
-		(end 66.9 44.58)
+		(end 66.41 44.09)
 		(width 0.5)
 		(layer "F.Cu")
