File: 01_Pcb/PLACA-GAMEBOY/PLACA-GAMEBOY.kicad_sch (KiCad schematic)
At the start: 8 parts, among them J1 Conn_01x08, SW1 SW_Push, SW2 SW_Push, SW3 SW_Push, SW4 SW_Push, SW5 SW_Push, SW6 SW_Push, U1 ESP32-S3-DEVKITC-1-N8R8

Commit message: document
Parts:
- added J2: Conn_01x02_Socket, TerminalBlock:TerminalBlock_MaiXu_MX126-5.0-02P_1x02_P5.00mm, symbol Connector:Conn_01x02_Socket
Connections:
- net at J1.7 (Pin_7), SW1.2, SW2.2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: now also J2.2 (Pin_2)
- net at SW3.1: now also U1.J1_5 (GPIO5); no longer U1.J1_4 (GPIO4)
- net at U1.J1_21 (5V0): now also J2.1 (Pin_1)
- net at SW4.1: now also U1.J1_4 (GPIO4); no longer U1.J1_5 (GPIO5)
- no-connect marks 30 -> 29
Other:
- moved on the sheet: SW3, SW6
